Commit message: robot.urdf: added links and joints for the 12 individual virtual distance sensors derived from laser scan

File: ros/robot.urdf (robot description, URDF)
Before this commit: robot robot, 9 links, 8 joints
Links:
- added link laser0
- added link laser1
- added link laser10
- added link laser11
- added link laser2
- added link laser3
- added link laser4
- added link laser5
- added link laser6
- added link laser7
- added link laser8
- added link laser9
Joints:
- added joint base_link_to_laser0: type fixed, parent base_link, child laser0, origin xyz=0.000 0.000 0.00 rpy=0 0 0
- added joint base_link_to_laser1: type fixed, parent base_link, child laser1, origin xyz=0.000 0.000 0.00 rpy=0 0 0.523599
- added joint base_link_to_laser10: type fixed, parent base_link, child laser10, origin xyz=0.000 0.000 0.00 rpy=0 0 5.235988
- added joint base_link_to_laser11: type fixed, parent base_link, child laser11, origin xyz=0.000 0.000 0.00 rpy=0 0 330
- added joint base_link_to_laser2: type fixed, parent base_link, child laser2, origin xyz=0.000 0.000 0.00 rpy=0 0 1.047198
- added joint base_link_to_laser3: type fixed, parent base_link, child laser3, origin xyz=0.000 0.000 0.00 rpy=0 0 1.570796
- added joint base_link_to_laser4: type fixed, parent base_link, child laser4, origin xyz=0.000 0.000 0.00 rpy=0 0 2.094395
- added joint base_link_to_laser5: type fixed, parent base_link, child laser5, origin xyz=0.000 0.000 0.00 rpy=0 0 2.617994
- added joint base_link_to_laser6: type fixed, parent base_link, child laser6, origin xyz=0.000 0.000 0.00 rpy=0 0 3.141593
- added joint base_link_to_laser7: type fixed, parent base_link, child laser7, origin xyz=0.000 0.000 0.00 rpy=0 0 3.665191
- added joint base_link_to_laser8: type fixed, parent base_link, child laser8, origin xyz=0.000 0.000 0.00 rpy=0 0 4.18879
- added joint base_link_to_laser9: type fixed, parent base_link, child laser9, origin xyz=0.000 0.000 0.00 rpy=0 0 4.712389

Commit message: robot.urdf: fixed typo

File: ros/robot.urdf (robot description, URDF)
Before this commit: robot robot, 21 links, 20 joints
Joints:
- joint base_link_to_laser11: origin xyz=0.000 0.000 0.00 rpy=0 0 330 -> xyz=0.000 0.000 0.00 rpy=0 0 5.759587

Commit message: robot.urdf:  add links and joints for the 12 virtual distance sensors

File: ros/robot.urdf (robot description, URDF)
Before this commit: robot robot, 21 links, 20 joints
Joints:
- joint base_link_to_laser1: origin xyz=0.000 0.000 0.00 rpy=0 0 0.523599 -> xyz=0.000 0.000 0.00 rpy=0 0 5.759587
- joint base_link_to_laser10: origin xyz=0.000 0.000 0.00 rpy=0 0 5.235988 -> xyz=0.000 0.000 0.00 rpy=0 0 1.047198
- joint base_link_to_laser11: origin xyz=0.000 0.000 0.00 rpy=0 0 5.759587 -> xyz=0.000 0.000 0.00 rpy=0 0 0.523599
- joint base_link_to_laser2: origin xyz=0.000 0.000 0.00 rpy=0 0 1.047198 -> xyz=0.000 0.000 0.00 rpy=0 0 5.235988
- joint base_link_to_laser3: origin xyz=0.000 0.000 0.00 rpy=0 0 1.570796 -> xyz=0.000 0.000 0.00 rpy=0 0 4.712389
- joint base_link_to_laser4: origin xyz=0.000 0.000 0.00 rpy=0 0 2.094395 -> xyz=0.000 0.000 0.00 rpy=0 0 4.18879
- joint base_link_to_laser5: origin xyz=0.000 0.000 0.00 rpy=0 0 2.617994 -> xyz=0.000 0.000 0.00 rpy=0 0 3.665191
- joint base_link_to_laser7: origin xyz=0.000 0.000 0.00 rpy=0 0 3.665191 -> xyz=0.000 0.000 0.00 rpy=0 0 2.617994
- joint base_link_to_laser8: origin xyz=0.000 0.000 0.00 rpy=0 0 4.18879 -> xyz=0.000 0.000 0.00 rpy=0 0 2.094395
- joint base_link_to_laser9: origin xyz=0.000 0.000 0.00 rpy=0 0 4.712389 -> xyz=0.000 0.000 0.00 rpy=0 0 1.570796
